Commit message: Fix URDF visualization launch

File: src/nxp_rs_description/urdf/nxp_rs.xacro (robot description, xacro)
@@ -1,3 +1,3 @@
-<?xml version="1.0">
+<?xml version="1.0"?>
 <robot name="nxp_rs" xmlns:xacro="http://www.ros.org/wiki/xacro">
     <link name="base_link">
@@ -5,13 +5,14 @@
             <origin xyz="0.00 0.00 0.00" rpy="0.00 0.00 0.00"/>
             <geometry>
-                <mesh filename="package://nxp_rs_description/meshes/base-link.stl"/>
+                <mesh filename="package://nxp_rs_description/meshes/base-link.STL"/>
             </geometry>
         </visual>
     </link>
     <joint name="joint-1" type="revolute">
-        <parent link="base-link"/>
-        <child link="link-1"/>
+        <parent link="base_link"/>
+        <child link="link_1"/>
         <origin xyz="0.00 0.00 0.06" rpy="0.00 0.00 0.00"/>
         <axis xyz="0 0 1"/>
+        <limit lower="-3.14159" upper="3.14159" effort="1.0" velocity="1.0"/>
     </joint>
     <link name="link_1">
@@ -19,13 +20,14 @@
             <origin xyz="0.00 0.00 0.00" rpy="0.00 0.00 0.00"/>
             <geometry>
-                <mesh filename="package://nxp_rs_description/meshes/link-1.stl"/>
+            <mesh filename="package://nxp_rs_description/meshes/link-1.STL"/>
             </geometry>
         </visual>
     </link>
     <joint name="joint-2" type="revolute">
-        <parent link="link-1"/>
-        <child link="link-2"/>
+        <parent link="link_1"/>
+        <child link="link_2"/>
         <origin xyz="0.00 -0.043 0.0445" rpy="0.00 0.00 0.00"/>
         <axis xyz="0 1 0"/>
+        <limit lower="-3.14159" upper="3.14159" effort="1.0" velocity="1.0"/>
     </joint>
     <link name="link_2">
@@ -33,13 +35,14 @@
             <origin xyz="0.00 0.00 0.00" rpy="0.00 0.00 0.00"/>
             <geometry>
-                <mesh filename="package://nxp_rs_description/meshes/link-2.stl"/>
+            <mesh filename="package://nxp_rs_description/meshes/link-2.STL"/>
             </geometry>
         </visual>
     </link>
     <joint name="joint-3" type="revolute">
-        <parent link="link-2"/>
-        <child link="link-3"/>
+        <parent link="link_2"/>
+        <child link="link_3"/>
         <origin xyz="0.00 0.046 0.1030" rpy="0.00 0.00 0.00"/>
         <axis xyz="0 0 1"/>
+        <limit lower="-3.14159" upper="3.14159" effort="1.0" velocity="1.0"/>
     </joint>
     <link name="link_3">
@@ -47,13 +50,14 @@
             <origin xyz="0.00 0.00 0.00" rpy="0.00 0.00 0.00"/>
             <geometry>
-                <mesh filename="package://nxp_rs_description/meshes/link-3.stl"/>
+            <mesh filename="package://nxp_rs_description/meshes/link-3.STL"/>
             </geometry>
         </visual>
     </link>
-    <joint name="joint-3" type="revolute">
-        <parent link="link-3"/>
-        <child link="link-4"/>
+    <joint name="joint-4" type="revolute">
+        <parent link="link_3"/>
+        <child link="link_4"/>
         <origin xyz="0.00 -0.043 0.0445" rpy="0.00 0.00 0.00"/>
         <axis xyz="0 1 0"/>
+        <limit lower="-3.14159" upper="3.14159" effort="1.0" velocity="1.0"/>
     </joint>
     <link name="link_4">
@@ -61,13 +65,14 @@
             <origin xyz="0.00 0.00 0.00" rpy="0.00 0.00 0.00"/>
             <geometry>
-                <mesh filename="package://nxp_rs_description/meshes/link-4.stl"/>
+            <mesh filename="package://nxp_rs_description/meshes/link-4.STL"/>
             </geometry>
         </visual>
     </link>
-    <joint name="joint-4" type="revolute">
-        <parent link="link-4"/>
-        <child link="link-5"/>
+    <joint name="joint-5" type="revolute">
+        <parent link="link_4"/>
+        <child link="link_5"/>
         <origin xyz="0.00 0.0125 0.095" rpy="0.00 0.00 0.00"/>
         <axis xyz="0 0 1"/>
+        <limit lower="-3.14159" upper="3.14159" effort="1.0" velocity="1.0"/>
     </joint>
     <link name="link_5">
@@ -75,13 +80,14 @@
             <origin xyz="0.00 0.00 0.00" rpy="0.00 0.00 0.00"/>
             <geometry>
-                <mesh filename="package://nxp_rs_description/meshes/link-5.stl"/>
+            <mesh filename="package://nxp_rs_description/meshes/link-5.STL"/>
             </geometry>
         </visual>
     </link>
-    <joint name="joint-5" type="revolute">
-        <parent link="link-5"/>
+    <joint name="joint-6" type="revolute">
+        <parent link="link_5"/>
         <child link="palm"/>
         <origin xyz="0.00 0.0322 0.0824" rpy="0.00 0.00 0.00"/>
         <axis xyz="0 1 0"/>
+        <limit lower="-3.14159" upper="3.14159" effort="1.0" velocity="1.0"/>
     </joint>
     <link name="palm">
@@ -89,5 +95,5 @@
             <origin xyz="0.00 0.00 0.00" rpy="0.00 0.00 0.00"/>
             <geometry>
-                <mesh filename="package://nxp_rs_description/meshes/palm.stl"/>
+            <mesh filename="package://nxp_rs_description/meshes/palm.STL"/>
             </geometry>
         </visual>
@@ -97,13 +103,14 @@
             <origin xyz="0.00 0.00 0.00" rpy="0.00 0.00 0.00"/>
             <geometry>
-                <mesh filename="package://nxp_rs_description/meshes/right-finger.stl"/>
+            <mesh filename="package://nxp_rs_description/meshes/right-finger.STL"/>
             </geometry>
         </visual>
     </link>
-    <joint name="joint_right-finger" type="linear">
+    <joint name="joint_right-finger" type="prismatic">
         <parent link="palm"/>
         <child link="right-finger"/>
         <origin xyz="-13.525 -77.126 60.400" rpy="0.00 0.00 0.00"/>
         <axis xyz="0 1 0"/>
+        <limit lower="-0.1" upper="0.1" effort="1.0" velocity="1.0"/>
     </joint>
     <link name="left-finger">
@@ -111,13 +118,14 @@
             <origin xyz="0.00 0.00 0.00" rpy="0.00 0.00 0.00"/>
             <geometry>
-                <mesh filename="package://nxp_rs_description/meshes/left-finger.stl"/>
+            <mesh filename="package://nxp_rs_description/meshes/left-finger.STL"/>
             </geometry>
         </visual>
     </link>
-    <joint name="joint_right-finger" type="linear">
+    <joint name="joint_left-finger" type="prismatic">
         <parent link="palm"/>
-        <child link="right-finger"/>
+        <child link="left-finger"/>
         <origin xyz="-13.525 77.126 60.400" rpy="0.00 0.00 0.00"/>
         <axis xyz="0 1 0"/>
+        <limit lower="-0.1" upper="0.1" effort="1.0" velocity="1.0"/>
     </joint>
 </robot>

Commit message: fixing mis-axis joint param

File: src/nxp_rs_description/urdf/nxp_rs.xacro (robot description, xacro)
@@ -73,5 +73,5 @@
         <child link="link_5"/>
         <origin xyz="0.00 0.0125 0.095" rpy="0.00 0.00 0.00"/>
-        <axis xyz="0 0 1"/>
+        <axis xyz="0 1 0"/>
         <limit lower="-3.14159" upper="3.14159" effort="1.0" velocity="1.0"/>
     </joint>
@@ -88,5 +88,5 @@
         <child link="palm"/>
         <origin xyz="0.00 0.0322 0.0824" rpy="0.00 0.00 0.00"/>
-        <axis xyz="0 1 0"/>
+        <axis xyz="0 0 1"/>
         <limit lower="-3.14159" upper="3.14159" effort="1.0" velocity="1.0"/>
     </joint>
@@ -110,5 +110,5 @@
         <parent link="palm"/>
         <child link="right-finger"/>
-        <origin xyz="-13.525 -77.126 60.400" rpy="0.00 0.00 0.00"/>
+        <origin xyz="-0.013525 -0.077126 0.060400" rpy="0.00 0.00 0.00"/>
         <axis xyz="0 1 0"/>
         <limit lower="-0.1" upper="0.1" effort="1.0" velocity="1.0"/>
@@ -125,5 +125,5 @@
         <parent link="palm"/>
         <child link="left-finger"/>
-        <origin xyz="-13.525 77.126 60.400" rpy="0.00 0.00 0.00"/>
+        <origin xyz="-0.013525 0.077126 0.060400" rpy="0.00 0.00 0.00"/>
         <axis xyz="0 1 0"/>
         <limit lower="-0.1" upper="0.1" effort="1.0" velocity="1.0"/>

Commit message: urdf fixed and moveit simulation demo

File: src/nxp_rs_description/urdf/nxp_rs.xacro (robot description, xacro)
@@ -1,11 +1,30 @@
 <?xml version="1.0"?>
 <robot name="nxp_rs" xmlns:xacro="http://www.ros.org/wiki/xacro">
+    <!-- Inertial data: meshes/*-inertial.txt, in kg, m and kg*m^2.
+         Use the L tensor about the COM, not the I tensor about the CAD origin.
+         Reports use positive products of inertia: negate off-diagonal L terms
+         for URDF. CAD output axes align with link axes except link_2 below.
+         Existing visual corrections already place meshes in these link frames;
+         do not apply those translations again to the reported COM. -->
     <link name="base_link">
         <visual>
-            <origin xyz="0.00 0.00 0.00" rpy="0.00 0.00 0.00"/>
+            <!-- STL mounting axis is at (20.710, 1.520, 0) mm. -->
+            <origin xyz="-0.020710 -0.001520 0.00" rpy="0.00 0.00 0.00"/>
             <geometry>
                 <mesh filename="package://nxp_rs_description/meshes/base-link.STL"/>
             </geometry>
         </visual>
+        <!-- SolidWorks: base-link-inertial.txt. -->
+        <inertial>
+            <origin xyz="0.000074 -0.000079 0.013768" rpy="0 0 0"/>
+            <mass value="0.370000"/>
+            <inertia ixx="0.000445" ixy="0.000001" ixz="-0.000001" iyy="0.000445" iyz="0.000001" izz="0.000672"/>
+        </inertial>
+        <collision>
+            <origin xyz="-0.020710 -0.001520 0.00" rpy="0.00 0.00 0.00"/>
+            <geometry>
+                <mesh filename="package://nxp_rs_description/meshes/base-link-col.STL"/>
+            </geometry>
+        </collision>
     </link>
     <joint name="joint-1" type="revolute">
@@ -23,4 +42,16 @@
             </geometry>
         </visual>
+        <!-- SolidWorks: link-1-inertial.txt. -->
+        <inertial>
+            <origin xyz="-0.000147 0.003478 0.032860" rpy="0 0 0"/>
+            <mass value="0.418000"/>
+            <inertia ixx="0.000433" ixy="0.000000" ixz="0.000001" iyy="0.000278" iyz="-0.000018" izz="0.000345"/>
+        </inertial>
+        <collision>
+            <origin xyz="0.00 0.00 0.00" rpy="0.00 0.00 0.00"/>
+            <geometry>
+                <mesh filename="package://nxp_rs_description/meshes/link-1-col.STL"/>
+            </geometry>
+        </collision>
     </link>
     <joint name="joint-2" type="revolute">
@@ -38,4 +69,19 @@
             </geometry>
         </visual>
+        <!-- SolidWorks: link-2-inertial.txt. -->
+        <!-- Inferred CAD-to-link rotation: Rx(pi), from STL COM and tensor.
+             Transform COM and tensor by R = diag(1, -1, -1).
+             Values below are expressed in the link frame (rpy = 0). -->
+        <inertial>
+            <origin xyz="-0.000157 0.044590 0.044463" rpy="0 0 0"/>
+            <mass value="0.405000"/>
+            <inertia ixx="0.000779" ixy="0.000000" ixz="0.000001" iyy="0.000508" iyz="-0.000003" izz="0.000458"/>
+        </inertial>
+        <collision>
+            <origin xyz="0.00 0.00 0.00" rpy="0.00 0.00 0.00"/>
+            <geometry>
+                <mesh filename="package://nxp_rs_description/meshes/link-2-col.STL"/>
+            </geometry>
+        </collision>
     </link>
     <joint name="joint-3" type="revolute">
@@ -53,4 +99,16 @@
             </geometry>
         </visual>
+        <!-- SolidWorks: link-3-inertial.txt. -->
+        <inertial>
+            <origin xyz="0.000004 0.003478 0.033003" rpy="0 0 0"/>
+            <mass value="0.418000"/>
+            <inertia ixx="0.000436" ixy="0.000000" ixz="0.000000" iyy="0.000280" iyz="-0.000018" izz="0.000343"/>
+        </inertial>
+        <collision>
+            <origin xyz="0.00 0.00 0.00" rpy="0.00 0.00 0.00"/>
+            <geometry>
+                <mesh filename="package://nxp_rs_description/meshes/link-3-col.STL"/>
+            </geometry>
+        </collision>
     </link>
     <joint name="joint-4" type="revolute">
@@ -63,9 +121,22 @@
     <link name="link_4">
     <visual>
-            <origin xyz="0.00 0.00 0.00" rpy="0.00 0.00 0.00"/>
+            <!-- STL lower pivot is at (24.240, 0, 20.200) mm. -->
+            <origin xyz="-0.024240 0.00 -0.020200" rpy="0.00 0.00 0.00"/>
             <geometry>
             <mesh filename="package://nxp_rs_description/meshes/link-4.STL"/>
             </geometry>
         </visual>
+        <!-- SolidWorks: link-4-inertial.txt. -->
+        <inertial>
+            <origin xyz="0.000000 0.046390 0.067030" rpy="0 0 0"/>
+            <mass value="0.260000"/>
+            <inertia ixx="0.000525" ixy="0.000000" ixz="0.000000" iyy="0.000378" iyz="-0.000004" izz="0.000219"/>
+        </inertial>
+        <collision>
+            <origin xyz="-0.024240 0.00 -0.020200" rpy="0.00 0.00 0.00"/>
+            <geometry>
+                <mesh filename="package://nxp_rs_description/meshes/link-4-col.STL"/>
+            </geometry>
+        </collision>
     </link>
     <joint name="joint-5" type="revolute">
@@ -78,9 +149,23 @@
     <link name="link_5">
     <visual>
-            <origin xyz="0.00 0.00 0.00" rpy="0.00 0.00 0.00"/>
+            <!-- STL pivot axis is offset by +23.230 mm along X. -->
+            <origin xyz="-0.023230 0.00 0.00" rpy="0.00 0.00 0.00"/>
             <geometry>
             <mesh filename="package://nxp_rs_description/meshes/link-5.STL"/>
             </geometry>
         </visual>
+        <!-- SolidWorks: link-5-inertial.txt. -->
+        <inertial>
+            <origin xyz="0.000002 0.032891 0.055468" rpy="0 0 0"/>
+            <mass value="0.237000"/>
+            <inertia ixx="0.000179" ixy="0.000000" ixz="0.000000" iyy="0.000127" iyz="0.000002" izz="0.000121"/>
+        </inertial>
+        <collision>
+            <!-- Collision STL is 17.675 mm higher than the visual STL. -->
+            <origin xyz="-0.023230 0.00 -0.017675" rpy="0.00 0.00 0.00"/>
+            <geometry>
+                <mesh filename="package://nxp_rs_description/meshes/link-5-col.STL"/>
+            </geometry>
+        </collision>
     </link>
     <joint name="joint-6" type="revolute">
@@ -93,17 +178,45 @@
     <link name="palm">
     <visual>
-            <origin xyz="0.00 0.00 0.00" rpy="0.00 0.00 0.00"/>
+            <!-- STL wrist mounting axis is at (16.463, 16.463, 0) mm. -->
+            <origin xyz="-0.016463 -0.016463 0.00" rpy="0.00 0.00 0.00"/>
             <geometry>
             <mesh filename="package://nxp_rs_description/meshes/palm.STL"/>
             </geometry>
         </visual>
+        <!-- SolidWorks: palm-inertial.txt. -->
+        <inertial>
+            <origin xyz="0.000001 -0.000001 0.042057" rpy="0 0 0"/>
+            <mass value="0.270000"/>
+            <inertia ixx="0.000232" ixy="0.000000" ixz="0.000000" iyy="0.000131" iyz="0.000000" izz="0.000178"/>
+        </inertial>
+        <collision>
+            <!-- Collision STL centre differs from the visual export origin. -->
+            <origin xyz="-0.0256281 -0.0778969 0.00" rpy="0.00 0.00 0.00"/>
+            <geometry>
+                <mesh filename="package://nxp_rs_description/meshes/palm-col.STL"/>
+            </geometry>
+        </collision>
     </link>
     <link name="right-finger">
     <visual>
-            <origin xyz="0.00 0.00 0.00" rpy="0.00 0.00 0.00"/>
+            <!-- Align STL to the supplied SolidWorks Coordinate System1:
+                 mounting plane Y = 12.0597 mm, X offset = 12.928 mm. -->
+            <origin xyz="-0.012928 -0.0120597 0.00" rpy="0.00 0.00 0.00"/>
             <geometry>
             <mesh filename="package://nxp_rs_description/meshes/right-finger.STL"/>
             </geometry>
         </visual>
+        <!-- SolidWorks: right-finger-inertial.txt. -->
+        <inertial>
+            <origin xyz="0.016200 0.014852 0.031385" rpy="0 0 0"/>
+            <mass value="0.033000"/>
+            <inertia ixx="0.000017" ixy="0.000000" ixz="0.000000" iyy="0.000021" iyz="-0.000003" izz="0.000011"/>
+        </inertial>
+        <collision>
+            <origin xyz="-0.012928 -0.0120597 0.00" rpy="0.00 0.00 0.00"/>
+            <geometry>
+                <mesh filename="package://nxp_rs_description/meshes/right-finger.STL"/>
+            </geometry>
+        </collision>
     </link>
     <joint name="joint_right-finger" type="prismatic">
@@ -116,9 +229,23 @@
     <link name="left-finger">
     <visual>
-            <origin xyz="0.00 0.00 0.00" rpy="0.00 0.00 0.00"/>
+            <!-- Align STL to the supplied SolidWorks Coordinate System1:
+                 mounting plane Y = 40.1475 mm, X offset = 12.928 mm. -->
+            <origin xyz="-0.012928 -0.0401475 0.00" rpy="0.00 0.00 0.00"/>
             <geometry>
             <mesh filename="package://nxp_rs_description/meshes/left-finger.STL"/>
             </geometry>
         </visual>
+        <!-- SolidWorks: left-finger-inertial.txt. -->
+        <inertial>
+            <origin xyz="0.016200 -0.014852 0.031385" rpy="0 0 0"/>
+            <mass value="0.033000"/>
+            <inertia ixx="0.000017" ixy="0.000000" ixz="0.000000" iyy="0.000021" iyz="0.000003" izz="0.000011"/>
+        </inertial>
+        <collision>
+            <origin xyz="-0.012928 -0.0401475 0.00" rpy="0.00 0.00 0.00"/>
+            <geometry>
+                <mesh filename="package://nxp_rs_description/meshes/left-finger.STL"/>
+            </geometry>
+        </collision>
     </link>
     <joint name="joint_left-finger" type="prismatic">
@@ -128,4 +255,6 @@
         <axis xyz="0 1 0"/>
         <limit lower="-0.1" upper="0.1" effort="1.0" velocity="1.0"/>
+        <!-- One physical actuator drives both mirrored fingers. -->
+        <mimic joint="joint_right-finger" multiplier="-1.0" offset="0.0"/>
     </joint>
 </robot>
