Commit message: Improve smooth jogging and motor calibration

File: src/nxp_rs_description/urdf/nxp_rs.xacro (robot description, xacro)
@@ -33,5 +33,5 @@
         <origin xyz="0.00 0.00 0.06" rpy="0.00 0.00 0.00"/>
         <axis xyz="0 0 1"/>
-        <limit lower="-3.14159" upper="3.14159" effort="1.0" velocity="1.0"/>
+        <limit lower="-3.238" upper="3.142" effort="1.0" velocity="1.0"/>
     </joint>
     <link name="link_1">
@@ -60,5 +60,5 @@
         <origin xyz="0.00 -0.043 0.0445" rpy="0.00 0.00 0.00"/>
         <axis xyz="0 1 0"/>
-        <limit lower="-3.14159" upper="3.14159" effort="1.0" velocity="1.0"/>
+        <limit lower="-1.863" upper="1.877" effort="1.0" velocity="1.0"/>
     </joint>
     <link name="link_2">
@@ -90,5 +90,5 @@
         <origin xyz="0.00 0.046 0.1030" rpy="0.00 0.00 0.00"/>
         <axis xyz="0 0 1"/>
-        <limit lower="-3.14159" upper="3.14159" effort="1.0" velocity="1.0"/>
+        <limit lower="-3.215" upper="3.015" effort="1.0" velocity="1.0"/>
     </joint>
     <link name="link_3">
@@ -117,5 +117,5 @@
         <origin xyz="0.00 -0.043 0.0445" rpy="0.00 0.00 0.00"/>
         <axis xyz="0 1 0"/>
-        <limit lower="-3.14159" upper="3.14159" effort="1.0" velocity="1.0"/>
+        <limit lower="-2.28" upper="2.086" effort="1.0" velocity="1.0"/>
     </joint>
     <link name="link_4">
@@ -145,5 +145,5 @@
         <origin xyz="0.00 0.0125 0.095" rpy="0.00 0.00 0.00"/>
         <axis xyz="0 1 0"/>
-        <limit lower="-3.14159" upper="3.14159" effort="1.0" velocity="1.0"/>
+        <limit lower="-1.839" upper="2.089" effort="1.0" velocity="1.0"/>
     </joint>
     <link name="link_5">
@@ -174,5 +174,5 @@
         <origin xyz="0.00 0.0322 0.0824" rpy="0.00 0.00 0.00"/>
         <axis xyz="0 0 1"/>
-        <limit lower="-3.14159" upper="3.14159" effort="1.0" velocity="1.0"/>
+        <limit lower="-3.24" upper="3.149" effort="1.0" velocity="1.0"/>
     </joint>
     <link name="palm">
@@ -225,5 +225,5 @@
         <origin xyz="-0.013525 -0.077126 0.060400" rpy="0.00 0.00 0.00"/>
         <axis xyz="0 1 0"/>
-        <limit lower="-0.1" upper="0.1" effort="1.0" velocity="1.0"/>
+        <limit lower="0.0" upper="0.0403" effort="1.0" velocity="1.0"/>
     </joint>
     <link name="left-finger">
@@ -254,5 +254,5 @@
         <origin xyz="-0.013525 0.077126 0.060400" rpy="0.00 0.00 0.00"/>
         <axis xyz="0 1 0"/>
-        <limit lower="-0.1" upper="0.1" effort="1.0" velocity="1.0"/>
+        <limit lower="-0.0403" upper="0.0" effort="1.0" velocity="1.0"/>
         <!-- One physical actuator drives both mirrored fingers. -->
         <mimic joint="joint_right-finger" multiplier="-1.0" offset="0.0"/>

File: src/nxp_rs_description/urdf/nxp_rs_mesh_only.xacro (robot description, xacro)
@@ -13,5 +13,5 @@
         <origin xyz="0.00 0.00 0.06" rpy="0.00 0.00 0.00"/>
         <axis xyz="0 0 1"/>
-        <limit lower="-3.14159" upper="3.14159" effort="1.0" velocity="1.0"/>
+        <limit lower="-3.238" upper="3.142" effort="1.0" velocity="1.0"/>
     </joint>
     <link name="link_1">
@@ -27,5 +27,5 @@
         <origin xyz="0.00 -0.043 0.0445" rpy="0.00 0.00 0.00"/>
         <axis xyz="0 1 0"/>
-        <limit lower="-3.14159" upper="3.14159" effort="1.0" velocity="1.0"/>
+        <limit lower="-1.863" upper="1.877" effort="1.0" velocity="1.0"/>
     </joint>
     <link name="link_2">
@@ -41,5 +41,5 @@
         <origin xyz="0.00 0.046 0.1030" rpy="0.00 0.00 0.00"/>
         <axis xyz="0 0 1"/>
-        <limit lower="-3.14159" upper="3.14159" effort="1.0" velocity="1.0"/>
+        <limit lower="-3.215" upper="3.015" effort="1.0" velocity="1.0"/>
     </joint>
     <link name="link_3">
@@ -55,5 +55,5 @@
         <origin xyz="0.00 -0.043 0.0445" rpy="0.00 0.00 0.00"/>
         <axis xyz="0 1 0"/>
-        <limit lower="-3.14159" upper="3.14159" effort="1.0" velocity="1.0"/>
+        <limit lower="-2.28" upper="2.086" effort="1.0" velocity="1.0"/>
     </joint>
     <link name="link_4">
@@ -69,5 +69,5 @@
         <origin xyz="0.00 0.0125 0.095" rpy="0.00 0.00 0.00"/>
         <axis xyz="0 1 0"/>
-        <limit lower="-3.14159" upper="3.14159" effort="1.0" velocity="1.0"/>
+        <limit lower="-1.839" upper="2.089" effort="1.0" velocity="1.0"/>
     </joint>
     <link name="link_5">
@@ -83,5 +83,5 @@
         <origin xyz="0.00 0.0322 0.0824" rpy="0.00 0.00 0.00"/>
         <axis xyz="0 0 1"/>
-        <limit lower="-3.14159" upper="3.14159" effort="1.0" velocity="1.0"/>
+        <limit lower="-3.24" upper="3.149" effort="1.0" velocity="1.0"/>
     </joint>
     <link name="palm">
@@ -104,5 +104,5 @@
         <origin xyz="-0.013525 -0.077126 0.060400" rpy="0.00 0.00 0.00"/>
         <axis xyz="0 1 0"/>
-        <limit lower="-0.1" upper="0.1" effort="1.0" velocity="1.0"/>
+        <limit lower="0.0" upper="0.0403" effort="1.0" velocity="1.0"/>
     </joint>
     <link name="left-finger">
@@ -118,5 +118,5 @@
         <origin xyz="-0.013525 0.077126 0.060400" rpy="0.00 0.00 0.00"/>
         <axis xyz="0 1 0"/>
-        <limit lower="-0.1" upper="0.1" effort="1.0" velocity="1.0"/>
+        <limit lower="-0.0403" upper="0.0" effort="1.0" velocity="1.0"/>
     </joint>
 </robot>

File: src/rs_control/urdf/nxp_rs_ros2_control.xacro (robot description, xacro)
@@ -25,4 +25,5 @@
       <state_interface name="velocity"/>
       <state_interface name="effort"/>
+      <state_interface name="temperature"/>
     </joint>
     <joint name="joint-2">
@@ -31,4 +32,5 @@
       <state_interface name="velocity"/>
       <state_interface name="effort"/>
+      <state_interface name="temperature"/>
     </joint>
     <joint name="joint-3">
@@ -37,4 +39,5 @@
       <state_interface name="velocity"/>
       <state_interface name="effort"/>
+      <state_interface name="temperature"/>
     </joint>
     <joint name="joint-4">
@@ -43,4 +46,5 @@
       <state_interface name="velocity"/>
       <state_interface name="effort"/>
+      <state_interface name="temperature"/>
     </joint>
     <joint name="joint-5">
@@ -49,4 +53,5 @@
       <state_interface name="velocity"/>
       <state_interface name="effort"/>
+      <state_interface name="temperature"/>
     </joint>
     <joint name="joint-6">
@@ -55,4 +60,5 @@
       <state_interface name="velocity"/>
       <state_interface name="effort"/>
+      <state_interface name="temperature"/>
     </joint>
     <joint name="joint_right-finger">
@@ -61,4 +67,5 @@
       <state_interface name="velocity"/>
       <state_interface name="effort"/>
+      <state_interface name="temperature"/>
     </joint>
   </ros2_control>

Commit message: done moveit

File: src/nxp_rs_description/urdf/nxp_rs.xacro (robot description, xacro)
@@ -24,5 +24,7 @@
             <origin xyz="-0.020710 -0.001520 0.00" rpy="0.00 0.00 0.00"/>
             <geometry>
-                <mesh filename="package://nxp_rs_description/meshes/base-link-col.STL"/>
+                <!-- Use the same detailed CAD mesh for visualisation and
+                     collision checking during commissioning. -->
+                <mesh filename="package://nxp_rs_description/meshes/base-link.STL"/>
             </geometry>
         </collision>
@@ -33,5 +35,5 @@
         <origin xyz="0.00 0.00 0.06" rpy="0.00 0.00 0.00"/>
         <axis xyz="0 0 1"/>
-        <limit lower="-3.238" upper="3.142" effort="1.0" velocity="1.0"/>
+        <limit lower="-3.14" upper="3.14" effort="1.0" velocity="1.0"/>
     </joint>
     <link name="link_1">
@@ -51,5 +53,5 @@
             <origin xyz="0.00 0.00 0.00" rpy="0.00 0.00 0.00"/>
             <geometry>
-                <mesh filename="package://nxp_rs_description/meshes/link-1-col.STL"/>
+                <mesh filename="package://nxp_rs_description/meshes/link-1.STL"/>
             </geometry>
         </collision>
@@ -81,5 +83,5 @@
             <origin xyz="0.00 0.00 0.00" rpy="0.00 0.00 0.00"/>
             <geometry>
-                <mesh filename="package://nxp_rs_description/meshes/link-2-col.STL"/>
+                <mesh filename="package://nxp_rs_description/meshes/link-2.STL"/>
             </geometry>
         </collision>
@@ -108,5 +110,5 @@
             <origin xyz="0.00 0.00 0.00" rpy="0.00 0.00 0.00"/>
             <geometry>
-                <mesh filename="package://nxp_rs_description/meshes/link-3-col.STL"/>
+                <mesh filename="package://nxp_rs_description/meshes/link-3.STL"/>
             </geometry>
         </collision>
@@ -136,5 +138,5 @@
             <origin xyz="-0.024240 0.00 -0.020200" rpy="0.00 0.00 0.00"/>
             <geometry>
-                <mesh filename="package://nxp_rs_description/meshes/link-4-col.STL"/>
+                <mesh filename="package://nxp_rs_description/meshes/link-4.STL"/>
             </geometry>
         </collision>
@@ -165,5 +167,5 @@
             <origin xyz="-0.023230 0.00 -0.017675" rpy="0.00 0.00 0.00"/>
             <geometry>
-                <mesh filename="package://nxp_rs_description/meshes/link-5-col.STL"/>
+                <mesh filename="package://nxp_rs_description/meshes/link-5.STL"/>
             </geometry>
         </collision>
@@ -194,8 +196,17 @@
             <origin xyz="-0.0256281 -0.0778969 0.00" rpy="0.00 0.00 0.00"/>
             <geometry>
-                <mesh filename="package://nxp_rs_description/meshes/palm-col.STL"/>
-            </geometry>
-        </collision>
-    </link>
+                <mesh filename="package://nxp_rs_description/meshes/palm.STL"/>
+            </geometry>
+        </collision>
+    </link>
+    <!-- Grasp/TCP frame: centered between the two finger CAD envelopes at
+         their open position. It is fixed to the palm, so the center remains
+         between the mirrored fingers as the gripper opens and closes. -->
+    <link name="grasp_frame"/>
+    <joint name="grasp_frame_joint" type="fixed">
+        <parent link="palm"/>
+        <child link="grasp_frame"/>
+        <origin xyz="0.002675 0.000000 0.103650" rpy="0.00 0.00 0.00"/>
+    </joint>
     <link name="right-finger">
     <visual>

File: src/nxp_rs_description/urdf/nxp_rs_mesh_only.xacro (robot description, xacro)
@@ -13,5 +13,5 @@
         <origin xyz="0.00 0.00 0.06" rpy="0.00 0.00 0.00"/>
         <axis xyz="0 0 1"/>
-        <limit lower="-3.238" upper="3.142" effort="1.0" velocity="1.0"/>
+        <limit lower="-3.14" upper="3.14" effort="1.0" velocity="1.0"/>
     </joint>
     <link name="link_1">
@@ -92,4 +92,11 @@
         </visual>
     </link>
+    <!-- Fixed grasp/TCP frame centered between the mirrored fingers. -->
+    <link name="grasp_frame"/>
+    <joint name="grasp_frame_joint" type="fixed">
+        <parent link="palm"/>
+        <child link="grasp_frame"/>
+        <origin xyz="0.002675 0.000000 0.103650" rpy="0.00 0.00 0.00"/>
+    </joint>
     <link name="right-finger">
     <visual>

File: src/rs_control/urdf/nxp_rs_ros2_control.xacro (robot description, xacro)
@@ -6,5 +6,5 @@
   <xacro:arg name="host_id" default="255"/>
   <xacro:arg name="response_timeout_ms" default="20"/>
-  <xacro:arg name="poll_rate_hz" default="20.0"/>
+  <xacro:arg name="poll_rate_hz" default="100.0"/>
   <xacro:arg name="read_only" default="true"/>
   <xacro:include filename="$(find nxp_rs_description)/urdf/nxp_rs.xacro"/>

Commit message: fix finger limit but still failed on joint 6 state sometimes

File: src/nxp_rs_description/urdf/nxp_rs.xacro (robot description, xacro)
@@ -176,5 +176,5 @@
         <origin xyz="0.00 0.0322 0.0824" rpy="0.00 0.00 0.00"/>
         <axis xyz="0 0 1"/>
-        <limit lower="-3.24" upper="3.149" effort="1.0" velocity="1.0"/>
+        <limit lower="-4.007354308" upper="2.381645692" effort="1.0" velocity="1.0"/>
     </joint>
     <link name="palm">
@@ -236,5 +236,5 @@
         <origin xyz="-0.013525 -0.077126 0.060400" rpy="0.00 0.00 0.00"/>
         <axis xyz="0 1 0"/>
-        <limit lower="0.0" upper="0.0403" effort="1.0" velocity="1.0"/>
+        <limit lower="0.0" upper="0.0837560613" effort="1.0" velocity="1.0"/>
     </joint>
     <link name="left-finger">
@@ -265,5 +265,5 @@
         <origin xyz="-0.013525 0.077126 0.060400" rpy="0.00 0.00 0.00"/>
         <axis xyz="0 1 0"/>
-        <limit lower="-0.0403" upper="0.0" effort="1.0" velocity="1.0"/>
+        <limit lower="-0.0837560613" upper="0.0" effort="1.0" velocity="1.0"/>
         <!-- One physical actuator drives both mirrored fingers. -->
         <mimic joint="joint_right-finger" multiplier="-1.0" offset="0.0"/>

File: src/nxp_rs_description/urdf/nxp_rs_mesh_only.xacro (robot description, xacro)
@@ -83,5 +83,5 @@
         <origin xyz="0.00 0.0322 0.0824" rpy="0.00 0.00 0.00"/>
         <axis xyz="0 0 1"/>
-        <limit lower="-3.24" upper="3.149" effort="1.0" velocity="1.0"/>
+        <limit lower="-4.007354308" upper="2.381645692" effort="1.0" velocity="1.0"/>
     </joint>
     <link name="palm">
@@ -111,5 +111,5 @@
         <origin xyz="-0.013525 -0.077126 0.060400" rpy="0.00 0.00 0.00"/>
         <axis xyz="0 1 0"/>
-        <limit lower="0.0" upper="0.0403" effort="1.0" velocity="1.0"/>
+        <limit lower="0.0" upper="0.0837560613" effort="1.0" velocity="1.0"/>
     </joint>
     <link name="left-finger">
@@ -125,5 +125,5 @@
         <origin xyz="-0.013525 0.077126 0.060400" rpy="0.00 0.00 0.00"/>
         <axis xyz="0 1 0"/>
-        <limit lower="-0.0403" upper="0.0" effort="1.0" velocity="1.0"/>
+        <limit lower="-0.0837560613" upper="0.0" effort="1.0" velocity="1.0"/>
     </joint>
 </robot>
